Commit message: added laser scan

File: SURover22_description_byerenna/urdf/SURover22_description_byerenna.urdf (robot description, URDF)
Before this commit: robot SURover22_description_byerenna, 7 links, 6 joints
Links:
- added link camera_link, mass 1e-5; collision box size=0.05 0.05 0.05; visual box size=0.05 0.05 0.05
Joints:
- added joint camera_joint: type fixed, parent base_link, child camera_link, origin xyz=0.05 0 0.3 rpy=0 0 0, axis 0 1 0
- joint joint-L-f: axis 0 -1 0 -> 0 1 0
- joint joint-L-m: axis 0 -1 0 -> 0 1 0
- joint joint-L-r: axis 0 -1 0 -> 0 1 0
- joint joint-R-f: axis 0 -1 0 -> 0 1 0
- joint joint-R-m: axis 0 -1 0 -> 0 1 0
- joint joint-R-r: axis 0 -1 0 -> 0 1 0

Commit message: error fixes

File: SURover22_description_byerenna/urdf/SURover22_description_byerenna.urdf (robot description, URDF)
Before this commit: robot SURover22_description_byerenna, 8 links, 7 joints
Joints:
- joint camera_joint: origin xyz=0.05 0 0.3 rpy=0 0 0 -> xyz=0.05 0 0.25 rpy=0 0 0

Commit message: Damla Commit

File: SURover22_description_byerenna/urdf/SURover22_description_byerenna.urdf (robot description, URDF)
Before this commit: robot SURover22_description_byerenna, 8 links, 7 joints
Joints:
- removed joint joint-L-f
- removed joint joint-L-m
- removed joint joint-L-r
- removed joint joint-R-f
- removed joint joint-R-m
- removed joint joint-R-r
- added joint joint_L_f: type continuous, parent base_link, child L-front, origin xyz=0.548812606572592 0.426079999999846 -0.428126101607028 rpy=0 0 0, axis 0 1 0
- added joint joint_L_m: type continuous, parent base_link, child L-mid, origin xyz=0.068429 0.46108 -0.42809 rpy=0 0 0, axis 0 1 0
- added joint joint_L_r: type continuous, parent base_link, child L-rear, origin xyz=-0.43564 0.46108 -0.42817 rpy=0 0 0, axis 0 1 0
- added joint joint_R_f: type continuous, parent base_link, child R-front, origin xyz=0.548838296645782 -0.351080000000064 -0.428087514508932 rpy=0 0 0, axis 0 1 0
- added joint joint_R_m: type continuous, parent base_link, child R-mid, origin xyz=0.068456 -0.38608 -0.42809 rpy=0 0 0, axis 0 1 0
- added joint joint_R_r: type continuous, parent base_link, child R-rear, origin xyz=-0.43561 -0.38608 -0.42822 rpy=0 0 0, axis 0 1 0
